File: LaserTransmitterReceivers/pcb/esp8266controllerPCB/esp8266controllerPCB.kicad_pcb (KiCad board)
At the start: 2 copper layers, 86 parts, among them J1 V-IN, J2 4, J3 5, J4 6, J5 7, J6 0, J7 1, J8 2, J9 3, Q1 85N3LHS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

Commit message: Update to version 1.0
Parts:
- added H1: MountingHole, MountingHole:MountingHole_6mm, F.Cu at (36.1, 90.9)
- added H2: MountingHole, MountingHole:MountingHole_6mm, F.Cu at (137.2, 90.9)
- added H3: MountingHole, MountingHole:MountingHole_6mm, F.Cu at (238.3, 90.9)
- moved R8 128.5 mm to (71.1, 106.7), turned to 180 degrees
- moved R9 126.9 mm to (88.3, 106.7), turned to 180 degrees
- moved C12 125.4 mm to (54.0, 116.2)
- moved C14 123.3 mm to (88.3, 116.2)
- moved D4 122.7 mm to (54.0, 104.1), turned to 180 degrees
- moved C6 121.7 mm to (97.8, 104.1), turned to 180 degrees
- moved JP2 121.4 mm to (59.1, 105.4)
- moved D5 120.7 mm to (71.1, 104.1), turned to 180 degrees
- moved D6 120.4 mm to (88.3, 104.1), turned to 180 degrees
- moved C13 119.1 mm to (71.1, 116.2)
- moved R4 117.1 mm to (81.3, 106.7), turned to 180 degrees
- moved C4 116.8 mm to (64.1, 104.1), turned to 180 degrees
- moved JP3 116.2 mm to (76.2, 105.4)
- moved D9 115.6 mm to (76.2, 116.2)
- moved C5 114.4 mm to (81.3, 104.1), turned to 180 degrees
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Routing:
- net /GND: track 0.00 -> 681.6 mm, vias 0 -> 57
- net /5V: track 0.00 -> 572.7 mm, vias 0 -> 9
- net /PORT3: track 0.00 -> 119.0 mm, vias 0 -> 1
- net /PORT2: track 0.00 -> 101.6 mm, vias 0 -> 1
- net /PORT1: track 0.00 -> 84.3 mm, vias 0 -> 1
- net /PORT4: track 0.00 -> 75.7 mm, vias 0 -> 1
- net /PORT0: track 0.00 -> 67.5 mm, vias 0 -> 1
- net /PORT5: track 0.00 -> 60.8 mm, vias 0 -> 1
- net /PORT6: track 0.00 -> 44.5 mm, vias 0 -> 1
- net Net-(C11-Pad2): track 0.00 -> 30.0 mm
- net Net-(C13-Pad2): track 0.00 -> 29.6 mm
- net Net-(C14-Pad2): track 0.00 -> 29.3 mm
- net Net-(C26-Pad2): track 0.00 -> 29.3 mm
- net Net-(C25-Pad2): track 0.00 -> 29.2 mm
- net Net-(C24-Pad2): track 0.00 -> 29.1 mm
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- added copper zone on B.Cu, net /GND
- added copper zone on F.Cu, net /GND
Other:
- board outline added: 224.2 x 60 mm
- board text added: "+ 6-30V"
- board text added: "-"
- board text added: "0"
- board text added: "1"
- board text added: "2"
- board text added: "3"
- board text added: "4"
- board text added: "5"
- board text added: "6"
- board text added: "7"
- board text added: "BOARD:"
- board text added: "ESP8266"
- board text added: "Lasermaze concentrator by PE1MEW pe1mew@gmail.com"
- board text added: "PORT"
- board text added: "POWER"
