File: LaserTransmitterReceivers/pcb/esp8266controllerPCB/esp8266controllerPCB.sch (KiCad schematic (older format))
At the start: 86 parts, among them J1 V-IN, J2 4, J3 5, J4 6, J5 7, J6 0, J7 1, J8 2, J9 3, Q1 85N3LHS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

Commit message: Update to version 1.0
Parts:
- added H1, H2, H3: MountingHole, MountingHole:MountingHole_6mm, symbol Mechanical:MountingHole
Changed lines of the file:
@@
 Text Notes 6100 5450 2    50   ~ 0
 Indicator output\nOptional control
+$Comp
+L Mechanical:MountingHole H1
+U 1 1 627B6DCB
+P 1600 4500
+F 0 "H1" H 1700 4546 50  0000 L CNN
+F 1 "MountingHole" H 1700 4455 50  0000 L CNN
+F 2 "MountingHole:MountingHole_6mm" H 1600 4500 50  0001 C CNN
+F 3 "~" H 1600 4500 50  0001 C CNN
+	1    1600 4500
+	1    0    0    -1
+$EndComp
+$Comp
+L Mechanical:MountingHole H2
+U 1 1 627B7188
+P 1600 4800
+F 0 "H2" H 1700 4846 50  0000 L CNN
+F 1 "MountingHole" H 1700 4755 50  0000 L CNN
+F 2 "MountingHole:MountingHole_6mm" H 1600 4800 50  0001 C CNN
+F 3 "~" H 1600 4800 50  0001 C CNN
+	1    1600 4800
+	1    0    0    -1
+$EndComp
+$Comp
+L Mechanical:MountingHole H3
+U 1 1 627B7E11
+P 1600 5100
+F 0 "H3" H 1700 5146 50  0000 L CNN
+F 1 "MountingHole" H 1700 5055 50  0000 L CNN
+F 2 "MountingHole:MountingHole_6mm" H 1600 5100 50  0001 C CNN
+F 3 "~" H 1600 5100 50  0001 C CNN
+	1    1600 5100
+	1    0    0    -1
+$EndComp
 $EndSCHEMATC
